File: adapter/386_adapter.kicad_sch (KiCad schematic)
At the start: 2 parts

Commit message: Add filter caps
Parts:
- added C1, C2: 100nF, Capacitor_SMD:C_1206_3216Metric_Pad1.33x1.80mm_HandSolder, symbol Device:C_Small
Connections:
- net GND: now also C1.2, C2.2
- net VCC: now also C1.1, C2.1
Changed lines of the file:
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@@
   (junction (at 208.28 17.78) (diameter 0) (color 0 0 0 0)
   )
+  (junction (at 134.62 180.34) (diameter 0) (color 0 0 0 0)
+  )
   (junction (at 218.44 160.02) (diameter 0) (color 0 0 0 0)
   )
@@
   )
   (junction (at 81.28 17.78) (diameter 0) (color 0 0 0 0)
+  )
+  (junction (at 134.62 172.72) (diameter 0) (color 0 0 0 0)
   )
   (junction (at 69.85 160.02) (diameter 0) (color 0 0 0 0)
@@
     (stroke (width 0) (type default))
   )
+  (wire (pts (xy 134.62 180.34) (xy 139.7 180.34))
+    (stroke (width 0) (type default))
+  )
   (wire (pts (xy 237.49 107.95) (xy 254 107.95))
     (stroke (width 0) (type default))
@@
     (stroke (width 0) (type default))
   )
+  (wire (pts (xy 128.27 180.34) (xy 134.62 180.34))
+    (stroke (width 0) (type default))
+  )
   (wire (pts (xy 96.52 17.78) (xy 96.52 21.59))
     (stroke (width 0) (type default))
@@
     (stroke (width 0) (type default))
   )
+  (wire (pts (xy 128.27 172.72) (xy 134.62 172.72))
+    (stroke (width 0) (type default))
+  )
   (wire (pts (xy 80.01 156.21) (xy 80.01 160.02))
     (stroke (width 0) (type default))
   )
+  (wire (pts (xy 139.7 180.34) (xy 139.7 179.07))
+    (stroke (width 0) (type default))
+  )
   (wire (pts (xy 215.9 17.78) (xy 218.44 17.78))
     (stroke (width 0) (type default))
@@
     (stroke (width 0) (type default))
   )
+  (wire (pts (xy 134.62 171.45) (xy 134.62 172.72))
+    (stroke (width 0) (type default))
+  )
   (wire (pts (xy 237.49 82.55) (xy 254 82.55))
     (stroke (width 0) (type default))
   )
+  (wire (pts (xy 128.27 179.07) (xy 128.27 180.34))
+    (stroke (width 0) (type default))
+  )
   (wire (pts (xy 237.49 31.75) (xy 254 31.75))
     (stroke (width 0) (type default))
@@
     (stroke (width 0) (type default))
   )
+  (wire (pts (xy 134.62 180.34) (xy 134.62 181.61))
+    (stroke (width 0) (type default))
+  )
   (wire (pts (xy 152.4 85.09) (xy 168.91 85.09))
     (stroke (width 0) (type default))
@@
     (stroke (width 0) (type default))
   )
+  (wire (pts (xy 139.7 172.72) (xy 139.7 173.99))
+    (stroke (width 0) (type default))
+  )
   (wire (pts (xy 114.3 52.07) (xy 130.81 52.07))
     (stroke (width 0) (type default))
   )
+  (wire (pts (xy 134.62 172.72) (xy 139.7 172.72))
+    (stroke (width 0) (type default))
+  )
   (wire (pts (xy 220.98 160.02) (xy 223.52 160.02))
     (stroke (width 0) (type default))
@@
   )
   (wire (pts (xy 91.44 17.78) (xy 91.44 21.59))
+    (stroke (width 0) (type default))
+  )
+  (wire (pts (xy 128.27 173.99) (xy 128.27 172.72))
     (stroke (width 0) (type default))
   )
@@
     )
   )
+  (symbol (lib_id "power:GND") (at 134.62 181.61 0) (unit 1)
+    (in_bom yes) (on_board yes) (dnp no) (fields_autoplaced)
+    (property "Reference" "#PWR05" (at 134.62 187.96 0)
+      (effects (font (size 1.27 1.27)) hide)
+    )
+    (property "Value" "GND" (at 134.62 186.69 0)
+      (effects (font (size 1.27 1.27)))
+    )
+    (property "Footprint" "" (at 134.62 181.61 0)
+      (effects (font (size 1.27 1.27)) hide)
+    )
+    (property "Datasheet" "" (at 134.62 181.61 0)
+      (effects (font (size 1.27 1.27)) hide)
+    )
+    (pin "1")
+    (instances
+      (project "386_adapter"
+        (path "/62869658-4f53-4ca4-98c2-2b0a91a7e94b"
+          (reference "#PWR05") (unit 1)
+        )
+      )
+    )
+  )
   (symbol (lib_id "power:GND") (at 81.28 161.29 0) (unit 1)
     (in_bom yes) (on_board yes) (dnp no) (fields_autoplaced)
@@
     )
   )
+  (symbol (lib_id "Device:C_Small") (at 139.7 176.53 0) (unit 1)
+    (in_bom yes) (on_board yes) (dnp no) (fields_autoplaced)
+    (property "Reference" "C2" (at 142.24 175.2663 0)
+      (effects (font (size 1.27 1.27)) (justify left))
+    )
+    (property "Value" "100nF" (at 142.24 177.8063 0)
+      (effects (font (size 1.27 1.27)) (justify left))
+    )
+    (property "Footprint" "Capacitor_SMD:C_1206_3216Metric_Pad1.33x1.80mm_HandSolder" (at 139.7 176.53 0)
+      (effects (font (size 1.27 1.27)) hide)
+    )
+    (property "Datasheet" "~" (at 139.7 176.53 0)
+      (effects (font (size 1.27 1.27)) hide)
+    )
+    (pin "1")
+    (pin "2")
+    (instances
+      (project "386_adapter"
+        (path "/62869658-4f53-4ca4-98c2-2b0a91a7e94b"
+          (reference "C2") (unit 1)
+        )
+      )
+    )
+  )
   (symbol (lib_id "power:GND") (at 204.47 161.29 0) (unit 1)
     (in_bom yes) (on_board yes) (dnp no) (fields_autoplaced)
@@
     )
   )
+  (symbol (lib_id "Device:C_Small") (at 128.27 176.53 0) (unit 1)
+    (in_bom yes) (on_board yes) (dnp no) (fields_autoplaced)
+    (property "Reference" "C1" (at 130.81 175.2663 0)
+      (effects (font (size 1.27 1.27)) (justify left))
+    )
+    (property "Value" "100nF" (at 130.81 177.8063 0)
+      (effects (font (size 1.27 1.27)) (justify left))
+    )
+    (property "Footprint" "Capacitor_SMD:C_1206_3216Metric_Pad1.33x1.80mm_HandSolder" (at 128.27 176.53 0)
+      (effects (font (size 1.27 1.27)) hide)
+    )
+    (property "Datasheet" "~" (at 128.27 176.53 0)
+      (effects (font (size 1.27 1.27)) hide)
+    )
+    (pin "1")
+    (pin "2")
+    (instances
+      (project "386_adapter"
+        (path "/62869658-4f53-4ca4-98c2-2b0a91a7e94b"
+          (reference "C1") (unit 1)
+        )
+      )
+    )
+  )
   (symbol (lib_id "power:VCC") (at 81.28 16.51 0) (unit 1)
     (in_bom yes) (on_board yes) (dnp no) (fields_autoplaced)
@@
         )
       )
+    )
+  )
+  (symbol (lib_id "power:VCC") (at 134.62 171.45 0) (unit 1)
+    (in_bom yes) (on_board yes) (dnp no) (fields_autoplaced)
+    (property "Reference" "#PWR06" (at 134.62 175.26 0)
+      (effects (font (size 1.27 1.27)) hide)
+    )
+    (property "Value" "VCC" (at 134.62 166.37 0)
+      (effects (font (size 1.27 1.27)))
+    )
+    (property "Footprint" "" (at 134.62 171.45 0)
+      (effects (font (size 1.27 1.27)) hide)
+    )
+    (property "Datasheet" "" (at 134.62 171.45 0)
+      (effects (font (size 1.27 1.27)) hide)
+    )
+    (pin "1")
+    (instances
+      (project "386_adapter"
+        (path "/62869658-4f53-4ca4-98c2-2b0a91a7e94b"
+          (reference "#PWR06") (unit 1)
+        )
+      )

Commit message: Update adapter for rev.3
Other:
- title: (none) -> 386DX QFP -> PGA Adapter
Changed lines of the file:
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@@
 	(generator_version "8.0")
 	(paper "A4")
+	(title_block
+		(title "386DX QFP -> PGA Adapter")
+		(rev "3")
+	)
 	(junction
 		(at 52.07 160.02)

Commit message: Some more changes for rev.3
Parts:
- U2: footprint Package_QFP:PQFP-132_24x24mm_P0.635mm_i386 -> Custom_QFP:PQFP-132_24x24mm_P0.635mm_i386
Changed lines of the file:
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@@
 			)
 		)
-		(property "Footprint" "Package_QFP:PQFP-132_24x24mm_P0.635mm_i386"
+		(property "Footprint" "Custom_QFP:PQFP-132_24x24mm_P0.635mm_i386"
 			(at 146.05 30.48 0)
 			(effects

Commit message: Update holder schematic and gerber
Changed lines of the file:
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@@
 		(on_board yes)
 		(dnp no)
-		(fields_autoplaced yes)
 		(property "Reference" "#PWR04"
 			(at 81.28 167.64 0)
@@
 		)
 		(property "Value" "GND"
-			(at 81.28 166.37 0)
+			(at 85.09 163.068 0)
 			(effects
 				(font
@@
 		(on_board yes)
 		(dnp no)
-		(fields_autoplaced yes)
 		(property "Reference" "#PWR02"
 			(at 205.74 20.32 0)
@@
 		)
 		(property "Value" "VCC"
-			(at 205.74 11.43 0)
+			(at 209.55 14.986 0)
 			(effects
 				(font
@@
 		(on_board yes)
 		(dnp no)
-		(fields_autoplaced yes)
 		(property "Reference" "#PWR03"
 			(at 204.47 167.64 0)
@@
 		)
 		(property "Value" "GND"
-			(at 204.47 166.37 0)
+			(at 208.788 163.068 0)
 			(effects
 				(font
@@
 		(on_board yes)
 		(dnp no)
-		(fields_autoplaced yes)
 		(property "Reference" "#PWR01"
 			(at 81.28 20.32 0)
@@
 		)
 		(property "Value" "VCC"
-			(at 81.28 11.43 0)
-			(effects
-				(font
+			(at 84.582 14.986 0)
+			(effects
+				(font
